Commit message: Updates 2/21
- Remove panel from xacro
- Create joint mask for purple and green
- Fix launching camera reference frames

File: wire_manipulation_description/urdf/environment.xacro (robot description, xacro)
@@ -2,5 +2,5 @@
 <robot xmlns:xacro="http://wiki.ros.org/xacro"
     name="environment">
-    <link name="panel_1">
+    <!-- <link name="panel_1">
         <visual>
             <origin xyz="0 0 0" rpy="0 0 0" />
@@ -35,6 +35,15 @@
             </geometry>
         </collision>
-    </link>
+    </link> -->
     <link name="ground">
+        <visual>
+            <origin xyz="0 0 0" rpy="0 0 0" />
+            <geometry>
+                <box size="5 5 0.02" />
+            </geometry>
+            <material name="Grey">
+                <color rgba="0.4 0.4 0.4 0.5" />
+            </material>
+        </visual>
         <collision>
             <origin xyz="0 0 0" rpy="0 0 0" />
@@ -44,5 +53,5 @@
         </collision>
     </link>
-    <joint name="panel_joint" type="fixed">
+    <!-- <joint name="panel_joint" type="fixed">
         <parent link="panel_1" />
         <child link="panel_2" />
@@ -53,5 +62,5 @@
         <child link="panel_1" />
         <origin xyz="0.5334 -0.0381 0.3048" />
-    </joint>
+    </joint> -->
     <joint name="ground_to_world" type="fixed">
         <parent link="world" />
